Commit message: Added the plugins for the camera, hokuyo and wheel joints

File: my_robot/urdf/my_robot.xacro (robot description, xacro)
@@ -1,4 +1,5 @@
 <?xml version='1.0'?>
 <robot name="my_robot" xmlns:xacro="http://www.ros.org/wiki/xacro">
+  <xacro:include filename="$(find my_robot)/urdf/my_robot.gazebo" />
   <link name="robot_footprint"></link>
   <joint name="robot_footprint_joint" type="fixed">
@@ -8,10 +9,11 @@
   </joint>
   <joint name="camera_joint" type="fixed">
-    <origin xyz="0.23 0 0" rpy="0 0 0"/>
+    <origin xyz="0.23 0 0.25" rpy="0 0 0"/>
     <parent link="chassis"/>
     <child link="camera"/>
+    <axis xyz="0 1 0"/>
   </joint>
   <joint name="hokuyo_joint" type="fixed">
-    <origin xyz="0.15 0 0.2" rpy="0 0 0" />
+    <origin xyz="0.15 0 0.32" rpy="0 0 0"/>
     <parent link="chassis"/>
     <child link="hokuyo" />
@@ -86,5 +88,5 @@
       </geometry>
       <material name="Yellow">
-         <color rgba="1 0.82 0 1.0"/>
+         <color rgba="1 0.82 0 1"/>
       </material>
     </visual>
@@ -101,5 +103,5 @@
       </geometry>
       <material name="Yellow">
-         <color rgba="1 0.82 0 1.0"/>
+         <color rgba="1 0.82 0 1"/>
       </material>
     </visual>
@@ -127,5 +129,5 @@
         <box size="0.1 0.18 0.2"/> </geometry>
       <material name="Yellow">
-         <color rgba="1 0.82 0 1.0"/>
+         <color rgba="1 0.82 0 1"/>
       </material>
     </visual>
@@ -151,5 +153,5 @@
       </geometry>
       <material name="Grey">
-         <color rgba="0.3 0.3 0.3 1.0"/>
+         <color rgba="0.3 0.3 0.3 1"/>
       </material>
     </visual>
@@ -175,5 +177,5 @@
       </geometry>
       <material name="Grey">
-         <color rgba="0.3 0.3 0.3 1.0"/>
+         <color rgba="0.3 0.3 0.3 1"/>
       </material>
     </visual>
@@ -199,5 +201,5 @@
       </geometry>
       <material name="Grey">
-         <color rgba="0.3 0.3 0.3 1.0"/>
+         <color rgba="0.3 0.3 0.3 1"/>
       </material>
     </visual>
@@ -223,5 +225,5 @@
       </geometry>
       <material name="Grey">
-         <color rgba="0.3 0.3 0.3 1.0"/>
+         <color rgba="0.3 0.3 0.3 1"/>
       </material>
     </visual>
@@ -247,5 +249,5 @@
       </geometry>
       <material name="Cyan">
-         <color rgba="0 1.0 1.0 1.0"/>
+         <color rgba="0 1 1 1"/>
       </material>
     </visual>
@@ -262,5 +264,5 @@
       </geometry>
       <material name="Cyan">
-         <color rgba="0 1.0 1.0 1.0"/>
+         <color rgba="0 1 1 1"/>
       </material>
     </visual>
@@ -277,5 +279,5 @@
       </geometry>
       <material name="Cyan">
-         <color rgba="0 1.0 1.0 1.0"/>
+         <color rgba="0 1 1 1"/>
       </material>
     </visual>

Commit message: Added bot to world. Made minor tweaks to improve robot movement

File: my_robot/urdf/my_robot.xacro (robot description, xacro)
@@ -42,5 +42,5 @@
     <axis xyz="0 1 0" rpy="0 0 0"/>
     <limit effort="10000" velocity="1000"/>
-    <dynamics damping="1.0" friction="1.0"/>
+    <dynamics damping="0" friction="0"/>
   </joint>
   <joint name="rear_left_wheel_hinge" type="continuous">
@@ -50,5 +50,5 @@
     <axis xyz="0 1 0" rpy="0 0 0"/>
     <limit effort="10000" velocity="1000"/>
-    <dynamics damping="1.0" friction="1.0"/>
+    <dynamics damping="0" friction="0"/>
   </joint>
   <joint name="arm_support_joint" type="fixed">

Commit message: Updated the model to help with wheel slippage

File: my_robot/urdf/my_robot.xacro (robot description, xacro)
@@ -26,5 +26,5 @@
     <axis xyz="0 1 0" rpy="0 0 0"/>
     <limit effort="10000" velocity="1000"/>
-    <dynamics damping="1.0" friction="1.0"/>
+    <dynamics damping="1.0" friction="5.0"/>
   </joint>
   <joint name="front_left_wheel_hinge" type="continuous">
@@ -34,5 +34,5 @@
     <axis xyz="0 1 0" rpy="0 0 0"/>
     <limit effort="10000" velocity="1000"/>
-    <dynamics damping="1.0" friction="1.0"/>
+    <dynamics damping="1.0" friction="5.0"/>
   </joint>
   <joint name="rear_right_wheel_hinge" type="continuous">
@@ -42,5 +42,5 @@
     <axis xyz="0 1 0" rpy="0 0 0"/>
     <limit effort="10000" velocity="1000"/>
-    <dynamics damping="0" friction="0"/>
+    <dynamics damping="1.0" friction="1.0"/>
   </joint>
   <joint name="rear_left_wheel_hinge" type="continuous">
@@ -50,5 +50,5 @@
     <axis xyz="0 1 0" rpy="0 0 0"/>
     <limit effort="10000" velocity="1000"/>
-    <dynamics damping="0" friction="0"/>
+    <dynamics damping="1.0" friction="1.0"/>
   </joint>
   <joint name="arm_support_joint" type="fixed">
@@ -268,5 +268,5 @@
     </visual>
     <collision name='bucket_collision'>
-      <origin xyz="0.36 0 0" rpy="0 0 0"/>
+      <origin xyz="0.36 0.1 0" rpy="0 0 0"/>
       <geometry>
         <box size="0.19 0.35 0.15"/>

Commit message: Fixed the torque and driving speeds.

File: my_robot/urdf/my_robot.xacro (robot description, xacro)
@@ -26,5 +26,5 @@
     <axis xyz="0 1 0" rpy="0 0 0"/>
     <limit effort="10000" velocity="1000"/>
-    <dynamics damping="1.0" friction="5.0"/>
+    <dynamics damping="1.0" friction="15.0"/>
   </joint>
   <joint name="front_left_wheel_hinge" type="continuous">
@@ -34,5 +34,5 @@
     <axis xyz="0 1 0" rpy="0 0 0"/>
     <limit effort="10000" velocity="1000"/>
-    <dynamics damping="1.0" friction="5.0"/>
+    <dynamics damping="1.0" friction="15.0"/>
   </joint>
   <joint name="rear_right_wheel_hinge" type="continuous">
@@ -42,5 +42,5 @@
     <axis xyz="0 1 0" rpy="0 0 0"/>
     <limit effort="10000" velocity="1000"/>
-    <dynamics damping="1.0" friction="1.0"/>
+    <dynamics damping="1.0" friction="0.5"/>
   </joint>
   <joint name="rear_left_wheel_hinge" type="continuous">
@@ -50,5 +50,5 @@
     <axis xyz="0 1 0" rpy="0 0 0"/>
     <limit effort="10000" velocity="1000"/>
-    <dynamics damping="1.0" friction="1.0"/>
+    <dynamics damping="1.0" friction="0.5"/>
   </joint>
   <joint name="arm_support_joint" type="fixed">

Commit message: Added proper Gazebo materials to my bot

File: my_robot/urdf/my_robot.xacro (robot description, xacro)
@@ -2,5 +2,5 @@
 <robot name="my_robot" xmlns:xacro="http://www.ros.org/wiki/xacro">
   <xacro:include filename="$(find my_robot)/urdf/my_robot.gazebo" />
-  <link name="robot_footprint"></link>
+  <!-- Joints -->
   <joint name="robot_footprint_joint" type="fixed">
     <origin xyz="0 0 0" rpy="0 0 0" />
@@ -42,5 +42,5 @@
     <axis xyz="0 1 0" rpy="0 0 0"/>
     <limit effort="10000" velocity="1000"/>
-    <dynamics damping="1.0" friction="0.5"/>
+    <dynamics damping="1.0" friction="15.0"/>
   </joint>
   <joint name="rear_left_wheel_hinge" type="continuous">
@@ -50,5 +50,5 @@
     <axis xyz="0 1 0" rpy="0 0 0"/>
     <limit effort="10000" velocity="1000"/>
-    <dynamics damping="1.0" friction="0.5"/>
+    <dynamics damping="1.0" friction="15.0"/>
   </joint>
   <joint name="arm_support_joint" type="fixed">
@@ -65,4 +65,6 @@
     <dynamics damping="1.0" friction="1.0"/>
   </joint>
+  <!-- Links-->
+  <link name="robot_footprint"></link>
   <link name='chassis'>
     <pose>0 0 0.1 0 0 0</pose>
@@ -87,7 +89,4 @@
         <box size="0.4 0.2 0.1"/>
       </geometry>
-      <material name="Yellow">
-         <color rgba="1 0.82 0 1"/>
-      </material>
     </visual>
     <collision name='cab_collision'>
@@ -102,7 +101,4 @@
         <box size="0.3 0.18 0.3"/>
       </geometry>
-      <material name="Yellow">
-         <color rgba="1 0.82 0 1"/>
-      </material>
     </visual>
   </link>
@@ -128,7 +124,4 @@
       <geometry>
         <box size="0.1 0.18 0.2"/> </geometry>
-      <material name="Yellow">
-         <color rgba="1 0.82 0 1"/>
-      </material>
     </visual>
   </link>
@@ -152,7 +145,4 @@
         <cylinder radius="0.1" length="0.05"/>
       </geometry>
-      <material name="Grey">
-         <color rgba="0.3 0.3 0.3 1"/>
-      </material>
     </visual>
   </link>
@@ -176,7 +166,4 @@
         <cylinder radius="0.1" length="0.05"/>
       </geometry>
-      <material name="Grey">
-         <color rgba="0.3 0.3 0.3 1"/>
-      </material>
     </visual>
   </link>
@@ -200,7 +187,4 @@
         <cylinder radius="0.1" length="0.05"/>
       </geometry>
-      <material name="Grey">
-         <color rgba="0.3 0.3 0.3 1"/>
-      </material>
     </visual>
   </link>
@@ -224,7 +208,4 @@
         <cylinder radius="0.1" length="0.05"/>
       </geometry>
-      <material name="Grey">
-         <color rgba="0.3 0.3 0.3 1"/>
-      </material>
     </visual>
   </link>
@@ -248,7 +229,4 @@
         <box size="0.58 0.01 0.04"/>
       </geometry>
-      <material name="Cyan">
-         <color rgba="0 1 1 1"/>
-      </material>
     </visual>
     <collision name='right_arm_collision'>
@@ -263,7 +241,4 @@
         <box size="0.58 0.01 0.04"/>
       </geometry>
-      <material name="Cyan">
-         <color rgba="0 1 1 1"/>
-      </material>
     </visual>
     <collision name='bucket_collision'>
@@ -278,7 +253,4 @@
         <box size="0.19 0.35 0.15"/>
       </geometry>
-      <material name="Cyan">
-         <color rgba="0 1 1 1"/>
-      </material>
     </visual>
   </link>
